File: kicad/stm32f103_FlyBoard_si4463/stm32f103_FlyBoard.kicad_sch (KiCad schematic)
At the start: 91 parts, among them J1 Conn_01x04_Male, J2 Conn_01x03_Male, J3 Conn_01x03_Male, J4 Conn_01x03_Male, J5 Conn_01x03_Male, J6 Conn_01x04_Male, J7 Conn_Coaxial, U1 STM32F103C8Tx, U2 MP2303ADN, U3 XC6206PxxxMR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

Commit message: after update cubemx
Parts:
- C13, C14: value 0.01u -> 10p
- C19: value 0.01u -> 8.2p
- C20: value 0.01u -> 13p
- C21: value 0.01u -> 3.9p
- C22: value 0.01u -> 2.2p
- C23, C29, C32: value 0.01u -> 9.1p
- C25, C26, C28: value 0.01u -> 56p
- C27, C31: value 0.01u -> 0.1u
- L2: value L -> 220n
- L3: value L -> 30n
- L4: value L -> 56n
- L5: value L -> 27n
- L6: value L -> 51n
- L7: value L -> 22n
- L8: value L -> 15n
- R1: value 1k -> 10k
- R20: value 100 -> 100 NC
- R8: value 0 -> 0 NC
- U6: value AS179-92LF -> PE4259
Other:
- note added: "Set this resistor for UART programming. (to SWDIO unset)"
- note added: "This resistor for 1S battery"
- note added: "Unset for 1S battery"
